Commit message: Fix the robot description
- Wheel separation 0.35 -> 0.376 m, measured from the meshes
- Lidar range 1.5 -> 12 m
- Move base_footprint to the drive axis
- Swap the IMU and dummy frames back
- Remove the ROS 1 control plugin and transmissions

File: testbed_description/urdf/testbed.xacro (robot description, xacro)
@@ -2,5 +2,4 @@
 <robot name="testbed" xmlns:xacro="http://www.ros.org/wiki/xacro">
 <xacro:include filename="$(find testbed_description)/urdf/materials.xacro" />
-<xacro:include filename="$(find testbed_description)/urdf/testbed.trans" />
 <xacro:include filename="$(find testbed_description)/urdf/testbed.gazebo" />
 <link name="base_footprint">
@@ -159,5 +158,5 @@
   </inertial>
   <visual>
-    <origin xyz="0.1 -0.05 -0.1612" rpy="0 0 0"/>
+    <origin xyz="0.0957 0.1238 -0.1595" rpy="0 0 0"/>
     <geometry>
       <mesh filename="file://$(find testbed_description)/meshes/imu_link_1.stl" scale="0.001 0.001 0.001"/>
@@ -166,5 +165,5 @@
   </visual>
   <collision>
-    <origin xyz="0.1 -0.05 -0.1612" rpy="0 0 0"/>
+    <origin xyz="0.0957 0.1238 -0.1595" rpy="0 0 0"/>
     <geometry>
       <mesh filename="file://$(find testbed_description)/meshes/imu_link_1.stl" scale="0.001 0.001 0.001"/>
@@ -179,5 +178,5 @@
   </inertial>
   <visual>
-    <origin xyz="0.1 0.14 -0.1612" rpy="0 0 0"/>
+    <origin xyz="0.0957 -0.0462 -0.1595" rpy="0 0 0"/>
     <geometry>
       <mesh filename="file://$(find testbed_description)/meshes/dummy_link_1.stl" scale="0.001 0.001 0.001"/>
@@ -186,5 +185,5 @@
   </visual>
   <collision>
-    <origin xyz="0.1 0.14 -0.1612" rpy="0 0 0"/>
+    <origin xyz="0.0957 -0.0462 -0.1595" rpy="0 0 0"/>
     <geometry>
       <mesh filename="file://$(find testbed_description)/meshes/dummy_link_1.stl" scale="0.001 0.001 0.001"/>
@@ -215,5 +214,5 @@
   <parent link="base_footprint" />
   <child link="base_link" />
-  <origin xyz="0 0 0" rpy="0 0 0" />
+  <origin xyz="0.0507 0.0379 0" rpy="0 0 0" />
 </joint>
 <joint name="left_wheel_joint" type="continuous">
@@ -249,10 +248,10 @@
 </joint>
 <joint name="imu_joint" type="fixed">
-  <origin xyz="-0.1 0.05 0.163" rpy="0 0 0"/>
+  <origin xyz="-0.0957 -0.1238 0.1595" rpy="0 0 0"/>
   <parent link="base_link"/>
   <child link="imu_link_1"/>
 </joint>
 <joint name="dummy_joint" type="fixed">
-  <origin xyz="-0.1 -0.1315 0.163" rpy="0 0 0"/>
+  <origin xyz="-0.0957 0.0462 0.1595" rpy="0 0 0"/>
   <parent link="base_link"/>
   <child link="dummy_link_1"/>
